File: boosterpack40.sch (KiCad schematic (older format))
At the start: 5 parts, among them J1 TI_BOOSTER_40_J1, J2 TI_BOOSTER_40_J2, J3 TI_BOOSTER_40_J3, J4 TI_BOOSTER_40_J4, J5 CONN_3

Commit message: добавлены документы
Parts:
- added P1: NRF24L01 MODUL, symbol CONN_4X2
Connections:
- net labels added: CE, CSN, IRO, MISO, MOSI, PD0, PD1, PD2, SCK
- wire segments 4 -> 15
Changed lines of the file:
@@
-EESchema Schematic File Version 2  date Thu 18 Oct 2012 10:04:05 PM PDT
+EESchema Schematic File Version 2
 LIBS:boosterpack
 LIBS:power
@@
 Sheet 1 1
 Title ""
-Date "19 oct 2012"
+Date "22 nov 2015"
 Rev ""
 Comp ""
@@
 F 0 "J5" V 7550 6800 50  0000 C CNN
 F 1 "CONN_3" V 7650 6800 40  0000 C CNN
+F 2 "" H 7600 6800 60  0001 C CNN
+F 3 "" H 7600 6800 60  0001 C CNN
 	1    7600 6800
 	1    0    0    1
 $EndComp
 Wire Wire Line
-	7250 6700 7000 6700
+	7000 6700 7250 6700
 Wire Wire Line
 	7250 6900 7000 6900
@@
 F 0 "#PWR01" H 7000 7000 30  0001 C CNN
 F 1 "VCC" H 7000 7000 30  0000 C CNN
+F 2 "" H 7000 6900 60  0001 C CNN
+F 3 "" H 7000 6900 60  0001 C CNN
 	1    7000 6900
 	0    -1   -1   0
@@
 F 0 "#PWR02" H 7000 6700 30  0001 C CNN
 F 1 "GND" H 7000 6630 30  0001 C CNN
+F 2 "" H 7000 6700 60  0001 C CNN
+F 3 "" H 7000 6700 60  0001 C CNN
 	1    7000 6700
 	0    1    1    0
@@
 F 0 "#PWR03" H 9150 2450 30  0001 C CNN
 F 1 "GND" H 9150 2380 30  0001 C CNN
+F 2 "" H 9150 2450 60  0001 C CNN
+F 3 "" H 9150 2450 60  0001 C CNN
 	1    9150 2450
 	0    1    1    0
@@
 F 0 "#PWR04" H 9150 1000 30  0001 C CNN
 F 1 "VCC" H 9150 1000 30  0000 C CNN
+F 2 "" H 9150 900 60  0001 C CNN
+F 3 "" H 9150 900 60  0001 C CNN
 	1    9150 900
 	0    -1   -1   0
@@
 F 0 "J1" H 9700 2000 60  0000 C CNN
 F 1 "TI_BOOSTER_40_J1" H 9750 700 60  0000 C CNN
+F 2 "" H 9750 1350 60  0001 C CNN
+F 3 "" H 9750 1350 60  0001 C CNN
 	1    9750 1350
 	1    0    0    -1
@@
 F 0 "J2" H 9700 3550 60  0000 C CNN
 F 1 "TI_BOOSTER_40_J2" H 9750 2250 60  0000 C CNN
+F 2 "" H 9750 2900 60  0001 C CNN
+F 3 "" H 9750 2900 60  0001 C CNN
 	1    9750 2900
 	1    0    0    -1
@@
 F 0 "J3" H 9700 5100 60  0000 C CNN
 F 1 "TI_BOOSTER_40_J3" H 9750 3800 60  0000 C CNN
+F 2 "" H 9750 4450 60  0001 C CNN
+F 3 "" H 9750 4450 60  0001 C CNN
 	1    9750 4450
 	1    0    0    -1
@@
 F 0 "J4" H 9700 6650 60  0000 C CNN
 F 1 "TI_BOOSTER_40_J4" H 9750 5350 60  0000 C CNN
+F 2 "" H 9750 6000 60  0001 C CNN
+F 3 "" H 9750 6000 60  0001 C CNN
 	1    9750 6000
 	1    0    0    -1
@@
 F 0 "#PWR05" H 9150 4100 30  0001 C CNN
 F 1 "GND" H 9150 4030 30  0001 C CNN
+F 2 "" H 9150 4100 60  0001 C CNN
+F 3 "" H 9150 4100 60  0001 C CNN
 	1    9150 4100
 	0    1    1    0
@@
 F 0 "#PWR06" H 9150 4090 20  0001 C CNN
 F 1 "+5V" H 9150 4090 30  0000 C CNN
+F 2 "" H 9150 4000 60  0001 C CNN
+F 3 "" H 9150 4000 60  0001 C CNN
 	1    9150 4000
 	0    -1   -1   0
 $EndComp
+$Comp
+L CONN_4X2 P1
+U 1 1 5651DDBB
+P 7450 1050
+F 0 "P1" H 7450 1300 50  0000 C CNN
+F 1 "NRF24L01 MODUL" H 7450 1400 40  0000 C CNN
+F 2 "" H 7450 1050 60  0000 C CNN
+F 3 "" H 7450 1050 60  0000 C CNN
+	1    7450 1050
+	1    0    0    -1
+$EndComp
+$Comp
+L GND #PWR07
+U 1 1 5651DEA5
+P 6850 900
+F 0 "#PWR07" H 6850 900 30  0001 C CNN
+F 1 "GND" H 6850 830 30  0001 C CNN
+F 2 "" H 6850 900 60  0000 C CNN
+F 3 "" H 6850 900 60  0000 C CNN
+	1    6850 900
+	0    1    1    0
+$EndComp
+Wire Wire Line
+	7050 900  6850 900
+$Comp
+L VCC #PWR08
+U 1 1 5651DF52
+P 8000 900
+F 0 "#PWR08" H 8000 1000 30  0001 C CNN
+F 1 "VCC" H 8000 1000 30  0000 C CNN
+F 2 "" H 8000 900 60  0000 C CNN
+F 3 "" H 8000 900 60  0000 C CNN
+	1    8000 900
+	1    0    0    -1
+$EndComp
+Wire Wire Line
+	7850 900  8000 900
+Text GLabel 8650 4200 0    60   Input ~ 0
+PD0
+Wire Wire Line
+	9150 4200 8650 4200
+Text GLabel 6750 1000 0    60   Input ~ 0
+CE
+Wire Wire Line
+	7050 1000 6750 1000
+Text GLabel 8900 4300 0    60   Input ~ 0
+PD1
+Wire Wire Line
+	9150 4300 8900 4300
+Text GLabel 8100 1000 2    60   3State ~ 0
+CSN
+Wire Wire Line
+	7850 1000 8100 1000
+Text GLabel 8650 4400 0    60   Input ~ 0
+PD2
+Wire Wire Line
+	9150 4400 8650 4400
+Text GLabel 7000 1100 0    60   Input ~ 0
+SCK
+Wire Wire Line
+	7050 1100 7000 1100
+Text GLabel 6750 1200 0    60   Output ~ 0
+MISO
+Wire Wire Line
+	7050 1200 6750 1200
+Text GLabel 8400 1100 2    60   Input ~ 0
+MOSI
+Wire Wire Line
+	7850 1100 8400 1100
+Text GLabel 7950 1200 2    60   Output ~ 0
+IRO
+Wire Wire Line
+	7850 1200 7950 1200
 $EndSCHEMATC
